Commit message: Adicionado urdf da base

File: catkin_ws/src/prototipo1/urdf/base.xacro (robot description, xacro)
@@ -1,27 +1,31 @@
 <?xml version="1.0"?>
+<!-- TODO medir parametros inerciais reais -->
 <robot xmlns:xacro="https://www.ros.org/wiki/xacro">
-	<link name="base_inferior">
+	<!-- Chutado -->
+	<xacro:property name="BASE_MASS" value="1"/>
+	<!-- Medidos -->
+	<xacro:property name="BASE_RADIUS" value="0.28"/>
+	<xacro:property name="BASE_THICKNESS" value="0.0155"/>
+	<link name="base_link">
 			<visual>
 					<geometry>
+							<cylinder length="${BASE_THICKNESS}" radius="${BASE_RADIUS}" />
 					</geometry>
-					<origin>
-					</origin>
-					<material>
-					</material>
+					<origin xyz="0 0 0.05" rpy="0 0 0" />
 			</visual>
 			<collision>
 					<geometry>
+						<cylinder length="${BASE_THICKNESS}" radius="${BASE_RADIUS}"/>
 					</geometry>
-					<origin>
-					</origin>
+					<origin xyz="0 0 0.05" rpy="0 0 0" />
 			</collision>
 			<inertial>
-					<mass>
-					</mass>
+					<mass value="${BASE_MASS}"/>
 					<!-- Centro de massa -->
-					<origin>
-					</origin>
-					<inertia>
-					</inertia>
+					<origin xyz="0 0 0" rpy="0 0 0"/>
+					<inertia
+							ixx="(1/12) * ${BASE_MASS} * (3 * ${BASE_RADIUS} * ${BASE_RADIUS} + ${BASE_THICKNESS} * ${BASE_THICKNESS})" ixy="0" ixz="0"
+							iyy="(1/12) * ${BASE_MASS} * (3 * ${BASE_RADIUS} * ${BASE_RADIUS} + ${BASE_THICKNESS} * ${BASE_THICKNESS})" iyz="0"
+							izz="(1/2) * ${BASE_MASS} * ${BASE_RADIUS} * ${BASE_RADIUS}"/>
 			</inertial>
 	</link>

Commit message: Can visualize robot xacro model in rviz. Adds a rviz config file.

File: catkin_ws/src/prototipo1/urdf/base.xacro (robot description, xacro)
@@ -3,5 +3,5 @@
 <robot xmlns:xacro="https://www.ros.org/wiki/xacro">
 	<!-- Chutado -->
-	<xacro:property name="BASE_MASS" value="1"/>
+	<xacro:property name="BASE_MASS" value="1.0"/>
 	<!-- Medidos -->
 	<xacro:property name="BASE_RADIUS" value="0.28"/>
@@ -25,7 +25,7 @@
 					<origin xyz="0 0 0" rpy="0 0 0"/>
 					<inertia
-							ixx="(1/12) * ${BASE_MASS} * (3 * ${BASE_RADIUS} * ${BASE_RADIUS} + ${BASE_THICKNESS} * ${BASE_THICKNESS})" ixy="0" ixz="0"
-							iyy="(1/12) * ${BASE_MASS} * (3 * ${BASE_RADIUS} * ${BASE_RADIUS} + ${BASE_THICKNESS} * ${BASE_THICKNESS})" iyz="0"
-							izz="(1/2) * ${BASE_MASS} * ${BASE_RADIUS} * ${BASE_RADIUS}"/>
+							ixx="${(1/12) * BASE_MASS * (3 * BASE_RADIUS * BASE_RADIUS + BASE_THICKNESS * BASE_THICKNESS)}" ixy="0" ixz="0"
+							iyy="${(1/12) * BASE_MASS * (3 * BASE_RADIUS * BASE_RADIUS + BASE_THICKNESS * BASE_THICKNESS)}" iyz="0"
+							izz="${(1/2) * BASE_MASS * BASE_RADIUS * BASE_RADIUS}"/>
 			</inertial>
 	</link>

File: catkin_ws/src/prototipo1/urdf/robot.urdf.xacro (robot description, xacro)
@@ -2,7 +2,7 @@
 <robot xmlns:xacro="http://www.ros.org/wiki/xacro" name="robot">
 		<xacro:include filename="base.xacro" />
-		<xacro:include filename="lidar.xacro" />
+		<!--<xacro:include filename="lidar.xacro" />
 		<xacro:include filename="camera.xacro" />
 		<xacro:include filename="motor_wheels.xacro" />
-		<xacro:include filename="joints.xacro" />
+		<xacro:include filename="joints.xacro" />-->
 </robot>

Commit message: Base + Support adicionados atualizados

File: catkin_ws/src/prototipo1/urdf/base.xacro (robot description, xacro)
@@ -25,7 +25,34 @@
 					<origin xyz="0 0 0" rpy="0 0 0"/>
 					<inertia
-							ixx="(1/12) * ${BASE_MASS} * (3 * ${BASE_RADIUS} * ${BASE_RADIUS} + ${BASE_THICKNESS} * ${BASE_THICKNESS})" ixy="0" ixz="0"
-							iyy="(1/12) * ${BASE_MASS} * (3 * ${BASE_RADIUS} * ${BASE_RADIUS} + ${BASE_THICKNESS} * ${BASE_THICKNESS})" iyz="0"
-							izz="(1/2) * ${BASE_MASS} * ${BASE_RADIUS} * ${BASE_RADIUS}"/>
+							ixx="${(1/12) * BASE_MASS * (3 * BASE_RADIUS * BASE_RADIUS + BASE_THICKNESS * BASE_THICKNESS)}" ixy="0" ixz="0"
+							iyy="${(1/12) * BASE_MASS * (3 * BASE_RADIUS * BASE_RADIUS + BASE_THICKNESS * BASE_THICKNESS)}" iyz="0"
+							izz="${(1/2) * BASE_MASS * BASE_RADIUS * BASE_RADIUS}"/>
+			</inertial>
+	</link>
+	<!-- Chutado -->
+    <xacro:property name="SUPPORT_MASS" value="0.5"/>
+    <!-- Medidos -->
+    <xacro:property name="SUPPORT_RADIUS" value="0.019"/>
+    <xacro:property name="SUPPORT_THICKNESS" value="1.25"/>
+	<link name="vertical_support_link">
+			<visual>
+				<geometry>
+						<cylinder length="${SUPPORT_THICKNESS}" radius="${SUPPORT_RADIUS}"/>
+				</geometry>
+				<origin xyz="0 0 -(1/2)*${SUPPORT_THICKNESS}" rpy="0 0 0"/>
+			</visual>
+			<collision>
+				<geometry>
+            			<cylinder length="${SUPPORT_THICKNESS}" radius="${SUPPORT_RADIUS}"/>
+            	</geometry>
+            	<origin xyz="0 0 -(1/2)*${SUPPORT_THICKNESS}" rpy="0 0 0"/>
+			</collision>
+			<inertial>
+					<mass value="${SUPPORT_MASS}"/>
+					<origin xyz="0 0 0" rpy="0 0 0"/>
+					<inertia
+                    		ixx="${(1/12) * SUPPORT_MASS * (3 * SUPPORT_RADIUS * SUPPORT_RADIUS +SUPPORT_THICKNESS * SUPPORT_THICKNESS)}" ixy="0" ixz="0"
+                    		iyy="${(1/12) * SUPPORT_MASS * (3 * SUPPORT_RADIUS * SUPPORT_RADIUS + SUPPORT_THICKNESS * SUPPORT_THICKNESS)}" iyz="0"
+                    		izz="${(1/2) * SUPPORT_MASS * SUPPORT_RADIUS * SUPPORT_RADIUS}"/>
 			</inertial>
 	</link>

File: catkin_ws/src/prototipo1/urdf/joints.xacro (robot description, xacro)
@@ -1,10 +1,14 @@
 <?xml version="1.0"?>
 <robot xmlns:xacro="http://www.ros.org/wiki/xacro" >
-        <joint name="base_inferior_lidar" type="fixed">
-            <parent link="base_inferior"/>
+		<!-- Joint to connect lidar to base
+        <joint name="base_lidar_joint" type="fixed">
+            <parent link="base_link"/>
             <child link="lidar"/>
             <origin xyz="" rpy=""/>
-            <axis xyz=""/>
-            <limit lower="" upper="" velocity="" effort="" />
-        </joint>
+		</joint> -->
+		<joint name="base_support_joint" type="fixed">
+				<parent link="base_link"/>
+				<parent link="support"/>
+				<origin xyz="0.205 0 ${(1/2)*BASE_THICKNESS}" rpy="0 0 0"/>
+		</joint>
 </robot>

Commit message: Fix z value of vertical_support_link. Failedd to insert color.

File: catkin_ws/src/prototipo1/urdf/base.xacro (robot description, xacro)
@@ -9,4 +9,7 @@
 	<link name="base_link">
 			<visual>
+					<material name="green">
+						<color rgba="0.2 1 0.2 1"/>
+					</material>
 					<geometry>
 							<cylinder length="${BASE_THICKNESS}" radius="${BASE_RADIUS}" />
@@ -40,5 +43,5 @@
 						<cylinder length="${SUPPORT_THICKNESS}" radius="${SUPPORT_RADIUS}"/>
 				</geometry>
-				<origin xyz="0 0 -(1/2)*${SUPPORT_THICKNESS}" rpy="0 0 0"/>
+				<origin xyz="0 0 ${(1/2)*SUPPORT_THICKNESS}" rpy="0 0 0"/>
 			</visual>
 			<collision>
@@ -46,5 +49,5 @@
             			<cylinder length="${SUPPORT_THICKNESS}" radius="${SUPPORT_RADIUS}"/>
             	</geometry>
-            	<origin xyz="0 0 -(1/2)*${SUPPORT_THICKNESS}" rpy="0 0 0"/>
+            	<origin xyz="0 0 ${(1/2)*SUPPORT_THICKNESS}" rpy="0 0 0"/>
 			</collision>
 			<inertial>

File: catkin_ws/src/prototipo1/urdf/joints.xacro (robot description, xacro)
@@ -9,6 +9,6 @@
 		<joint name="base_support_joint" type="fixed">
 				<parent link="base_link"/>
-				<parent link="vertical_support_link"/>
-				<origin xyz="0.205 0 ${(1/2)*BASE_THICKNESS}" rpy="0 0 0"/>
+				<child link="vertical_support_link"/>
+				<origin xyz="0.205 0 ${(1/2)*BASE_THICKNESS + 0.05}" rpy="0 0 0"/>
 		</joint>
 </robot>

File: catkin_ws/src/prototipo1/urdf/robot.urdf.xacro (robot description, xacro)
@@ -4,5 +4,5 @@
 		<!--<xacro:include filename="lidar.xacro" />
 		<xacro:include filename="camera.xacro" />
-		<xacro:include filename="motor_wheels.xacro" />
-		<xacro:include filename="joints.xacro" />-->
+		<xacro:include filename="motor_wheels.xacro" /> -->
+		<xacro:include filename="joints.xacro" />
 </robot>

Commit message: Completada descricao do prototipo1 em URDF. Para visualizar, apenas de rosrun no launch file rviz_test_urdf_gui.launch, mude o frame estático para base_link (ao invés de map), e, para melhor visualização, adicione um campo para ver os tf's

File: catkin_ws/src/prototipo1/urdf/base.xacro (robot description, xacro)
@@ -2,30 +2,40 @@
 <!-- TODO medir parametros inerciais reais -->
 <robot xmlns:xacro="https://www.ros.org/wiki/xacro">
+	<material name="gray">
+  		<color rgba="0.5 0.5 0.5 1"/>
+  	</material>
+	<material name="white">
+  		<color rgba="1 1 1 1"/>
+  	</material>
 	<!-- Chutado -->
-	<xacro:property name="BASE_MASS" value="1.0"/>
+	<xacro:property name="CHASSI_MASS" value="1.0"/>
 	<!-- Medidos -->
-	<xacro:property name="BASE_RADIUS" value="0.28"/>
-	<xacro:property name="BASE_THICKNESS" value="0.0155"/>
-	<link name="base_link">
+	<xacro:property name="CHASSI_RADIUS" value="0.28"/>
+	<xacro:property name="CHASSI_THICKNESS" value="0.0155"/>
+	<!-- Virtual base as recommended -->
+	<link name="base_link"/>
+	<!-- Real base, named as chassi -->
+	<link name="chassi_link">
 			<visual>
 					<geometry>
-							<cylinder length="${BASE_THICKNESS}" radius="${BASE_RADIUS}" />
+							<cylinder length="${CHASSI_THICKNESS}" radius="${CHASSI_RADIUS}" />
 					</geometry>
-					<origin xyz="0 0 0.05" rpy="0 0 0" />
+					<origin xyz="0 0 0" rpy="0 0 0" />
+					<material name="white"/>
 			</visual>
 			<collision>
 					<geometry>
-						<cylinder length="${BASE_THICKNESS}" radius="${BASE_RADIUS}"/>
+						<cylinder length="${CHASSI_THICKNESS}" radius="${CHASSI_RADIUS}"/>
 					</geometry>
-					<origin xyz="0 0 0.05" rpy="0 0 0" />
+					<origin xyz="0 0 0" rpy="0 0 0" />
 			</collision>
 			<inertial>
-					<mass value="${BASE_MASS}"/>
+					<mass value="${CHASSI_MASS}"/>
 					<!-- Centro de massa -->
 					<origin xyz="0 0 0" rpy="0 0 0"/>
 					<inertia
-							ixx="${(1/12) * BASE_MASS * (3 * BASE_RADIUS * BASE_RADIUS + BASE_THICKNESS * BASE_THICKNESS)}" ixy="0" ixz="0"
-							iyy="${(1/12) * BASE_MASS * (3 * BASE_RADIUS * BASE_RADIUS + BASE_THICKNESS * BASE_THICKNESS)}" iyz="0"
-							izz="${(1/2) * BASE_MASS * BASE_RADIUS * BASE_RADIUS}"/>
+							ixx="${(1/12) * CHASSI_MASS * (3 * CHASSI_RADIUS * CHASSI_RADIUS + CHASSI_THICKNESS * CHASSI_THICKNESS)}" ixy="0" ixz="0"
+							iyy="${(1/12) * CHASSI_MASS * (3 * CHASSI_RADIUS * CHASSI_RADIUS + CHASSI_THICKNESS * CHASSI_THICKNESS)}" iyz="0"
+							izz="${(1/2) * CHASSI_MASS * CHASSI_RADIUS * CHASSI_RADIUS}"/>
 			</inertial>
 	</link>
@@ -40,5 +50,6 @@
 						<cylinder length="${SUPPORT_THICKNESS}" radius="${SUPPORT_RADIUS}"/>
 				</geometry>
-				<origin xyz="0 0 -(1/2)*${SUPPORT_THICKNESS}" rpy="0 0 0"/>
+				<origin xyz="0 0 ${(1/2) * SUPPORT_THICKNESS}" rpy="0 0 0"/>
+				<material name="gray"/>
 			</visual>
 			<collision>
@@ -46,5 +57,5 @@
             			<cylinder length="${SUPPORT_THICKNESS}" radius="${SUPPORT_RADIUS}"/>
             	</geometry>
-            	<origin xyz="0 0 -(1/2)*${SUPPORT_THICKNESS}" rpy="0 0 0"/>
+            	<origin xyz="0 0 ${(1/2) * SUPPORT_THICKNESS}" rpy="0 0 0"/>
 			</collision>
 			<inertial>

File: catkin_ws/src/prototipo1/urdf/joints.xacro (robot description, xacro)
@@ -1,14 +1,48 @@
 <?xml version="1.0"?>
-<robot xmlns:xacro="http://www.ros.org/wiki/xacro" >
-		<!-- Joint to connect lidar to base
-        <joint name="base_lidar_joint" type="fixed">
-            <parent link="base_link"/>
-            <child link="lidar"/>
-            <origin xyz="" rpy=""/>
-		</joint> -->
-		<joint name="base_support_joint" type="fixed">
-				<parent link="base_link"/>
-				<parent link="support"/>
-				<origin xyz="0.205 0 ${(1/2)*BASE_THICKNESS}" rpy="0 0 0"/>
+<robot xmlns:xacro="http://www.ros.org/wiki/xacro">
+	<!-- Constants-->
+	<xacro:property name="PI" value="3.14159" />
+	<!-- Joint distance parameters -->
+	<xacro:property name="CAMERA_HEIGHT" value="${(4/5)*SUPPORT_THICKNESS}" />
+	<xacro:property name="BASE_LIDAR_DIST" value="0.2" />
+	<xacro:property name="BASE_WHEEL_DIST" value="0.28" />
+	<xacro:property name="BASE_SUPPORT_DIST" value="0.205" />
+	<xacro:property name="CHASSI_HEIGHT" value="0.05" />
+	<!-- To connect virtual (center of rotation) base to real one (chassi) -->
+	<joint name="base_chassi_joint" type="fixed">
+		<parent link="base_link" />
+		<child link="chassi_link" />
+		<origin xyz="-0.001 0 0" rpy="0 0 0" />
+	</joint>
+	<joint name="base_support_joint" type="fixed">
+		<parent link="base_link" />
+		<child link="vertical_support_link" />
+		<origin xyz="${-BASE_SUPPORT_DIST} 0 ${(1/2)*CHASSI_THICKNESS}" rpy="0 0 0" />
+	</joint>
+	<!-- By the conventions of ROS urdf/tf, left side is positive y axis, as so, side parameter is 1 if left, -1 if right-->
+	<xacro:macro name="wheel_joint" params="position_prefix side">
+		<joint name="${position_prefix}_wheel_joint" type="continuous">
+			<parent link="base_link" />
+			<child link="${position_prefix}_wheel_link" />
+			<!-- Adjust position based on the side that's on-->
+			<origin xyz="0 ${side*BASE_WHEEL_DIST} 0" rpy="${-(1/2)*PI*side} 0 0" />
+			<!-- Positive around counterclockwise z-axis -->
+			<axis xyz="0 0 ${side}" />
 		</joint>
+	</xacro:macro>
+	<!-- Define actual joints-->
+	<xacro:wheel_joint position_prefix="left" side="1" />
+	<xacro:wheel_joint position_prefix="right" side="-1" />
+	<!-- Joint to connect lidar to base -->
+	<joint name="base_lidar_joint" type="fixed">
+		<parent link="base_link" />
+		<child link="lidar_link" />
+		<origin xyz="${BASE_LIDAR_DIST} 0 ${(1/2)*CHASSI_THICKNESS}" rpy="0 0 0" />
+	</joint>
+	<!-- Joint to connect camera to support -->
+	<joint name="vertical_support_camera_joint" type="fixed">
+		<parent link="vertical_support_link" />
+		<child link="camera_link" />
+		<origin xyz="${SUPPORT_RADIUS} 0 ${CAMERA_HEIGHT}" rpy="${PI/2} 0 0" />
+	</joint>
 </robot>

File: catkin_ws/src/prototipo1/urdf/motor_wheels.xacro (robot description, xacro)
@@ -1,29 +1,39 @@
 <?xml version="1.0"?>
-<robot xmlns="http://www.ros.org/wiki/xacro">
-		<property name="PI" value="3.14159"/>
-		<!-- Wheel Properties -->
-   		<xacro:property name="wheel_base" value="" />
-    	<xacro:property name="wheel_track" value="" />
-    	<xacro:property name="wheel_vertical_offset" value="" />
-    	<xacro:property name="wheel_width" value="" />
-   		<xacro:property name="wheel_radius" value="" />
-    	<xacro:property name="wheel_mass" value="" />
-		<xacro:macro name="wheel_${position_sufffix}_joint" params="position_suffix ">
-		</xacro:macro>
-		<xacro:macro name="generic_wheel" params="position_prefix lado proa">
-        	<link name="${position_fixed}_wheel">
-           		<visual>
-                	<origin xyz="${lado*wheel_radius} ${-lado*wheel_width/2} ${-wheel_radius}" rpy="${PI/2} 0 ${lado*PI/2+PI/2}" />
-            	</visual>
-            	<collision>
-               		<geometry></geometry>
-                	<origin></origin>
-            	</collision>
-            	<inertial>
-                	<mass></mass>
-                	<origin></origin>
-                	<inertia></inertia>
-            	</inertial>
-        	</link>
-    	</xacro:macro>
+<robot xmlns:xacro="http://www.ros.org/wiki/xacro">
+	<material name="black">
+		<color rgba="0 0 0 1"/>
+	</material>
+	<!-- Wheel Properties -->
+	<xacro:property name="WHEEL_THICKNESS" value="0.051" />
+	<xacro:property name="WHEEL_RADIUS" value="0.08" />
+	<!-- Chutado -->
+	<xacro:property name="WHEEL_MASS" value="1" />
+	<xacro:macro name="wheel_link" params="position_prefix">
+		<link name="${position_prefix}_wheel_link">
+			<visual>
+				<geometry>
+					<cylinder length="${WHEEL_THICKNESS}" radius="${WHEEL_RADIUS}" />
+				</geometry>
+				<!--
+				<origin xyz="0 0 ${(1/2)*WHEEL_THICKNESS}" rpy="0 0 0" />
+				-->
+				<origin xyz="0 0 0" rpy="0 0 0" />
+				<material name="black" />
+			</visual>
+			<collision>
+				<geometry>
+					<cylinder length="${WHEEL_THICKNESS}" radius="${WHEEL_RADIUS}" />
+				</geometry>
+				<origin xyz="0 0 0" rpy="0 0 0" />
+			</collision>
+			<inertial>
+				<mass value="${WHEEL_MASS}" />
+				<!-- Centro de massa -->
+				<origin xyz="0 0 0" rpy="0 0 0" />
+				<inertia ixx="${(1/12) * WHEEL_MASS * (3 * WHEEL_RADIUS * WHEEL_RADIUS + WHEEL_THICKNESS * WHEEL_THICKNESS)}" ixy="0" ixz="0" iyy="${(1/12) * WHEEL_MASS * (3 * WHEEL_RADIUS * WHEEL_RADIUS + WHEEL_THICKNESS * WHEEL_THICKNESS)}" iyz="0" izz="${(1/2) * WHEEL_MASS * WHEEL_RADIUS * WHEEL_RADIUS}" />
+			</inertial>
+		</link>
+	</xacro:macro>
+	<xacro:wheel_link position_prefix="left" />
+	<xacro:wheel_link position_prefix="right" />
 </robot>

File: catkin_ws/src/prototipo1/urdf/robot.urdf.xacro (robot description, xacro)
@@ -2,7 +2,7 @@
 <robot xmlns:xacro="http://www.ros.org/wiki/xacro" name="robot">
 		<xacro:include filename="base.xacro" />
-		<!--<xacro:include filename="lidar.xacro" />
+		<xacro:include filename="lidar.xacro" />
 		<xacro:include filename="camera.xacro" />
 		<xacro:include filename="motor_wheels.xacro" />
-		<xacro:include filename="joints.xacro" />-->
+		<xacro:include filename="joints.xacro" />
 </robot>

Commit message: Errinho na cor

File: catkin_ws/src/prototipo1/urdf/base.xacro (robot description, xacro)
@@ -18,7 +18,4 @@
 	<link name="chassi_link">
 			<visual>
-					<material name="green">
-						<color rgba="0.2 1 0.2 1"/>
-					</material>
 					<geometry>
 							<cylinder length="${CHASSI_THICKNESS}" radius="${CHASSI_RADIUS}" />
