Commit message: Error in camera_imu_optical_frame. Made some changes in urdf files that maybe need to be reversed.

File: catkin_ws/src/prototipo1/urdf/camera.xacro (robot description, xacro)
@@ -6,5 +6,5 @@
 	<xacro:property name="CAMERA_RADIUS" value="0.05"/>
 	<xacro:property name="CAMERA_THICKNESS" value="0.1"/>
-	<link name="camera_link">
+	<link name="camera_imu_optical_frame">
 			<visual>
 					<geometry>

File: catkin_ws/src/prototipo1/urdf/joints.xacro (robot description, xacro)
@@ -58,5 +58,5 @@
 	<joint name="vertical_support_camera_joint" type="fixed">
 		<parent link="vertical_support_link" />
-		<child link="camera_link" />
+		<child link="camera_imu_optical_frame" />
 		<origin xyz="${SUPPORT_RADIUS} 0 ${CAMERA_HEIGHT}" rpy="${PI/2} 0 0" />
 	</joint>

Commit message: Added motor parameters according to model got with data analysis in matlab, used continuos transfer function with 4 poles and one zero. Parameters only correct for left side fn

File: catkin_ws/src/prototipo1/urdf/camera.xacro (robot description, xacro)
@@ -6,5 +6,5 @@
 	<xacro:property name="CAMERA_RADIUS" value="0.05"/>
 	<xacro:property name="CAMERA_THICKNESS" value="0.1"/>
-	<link name="camera_imu_optical_frame">
+	<link name="camera_link">
 			<visual>
 					<geometry>

File: catkin_ws/src/prototipo1/urdf/joints.xacro (robot description, xacro)
@@ -58,6 +58,12 @@
 	<joint name="vertical_support_camera_joint" type="fixed">
 		<parent link="vertical_support_link" />
-		<child link="camera_imu_optical_frame" />
+		<child link="camera_link" />
 		<origin xyz="${SUPPORT_RADIUS} 0 ${CAMERA_HEIGHT}" rpy="${PI/2} 0 0" />
 	</joint>
+	<!-- Connect unified IMU link to camera_link
+	<joint name="imu_joint" type="fixed">
+		<parent link="camera_link" />
+		<child link="camera_imu_optical_frame" />
+		<origin xyz="0 0 0" rpy="0 0 0" />
+	</joint> -->
 </robot>

Commit message: Trying to tune IMU and sensor fusion

File: catkin_ws/src/prototipo1/urdf/camera.xacro (robot description, xacro)
@@ -30,3 +30,5 @@
 			</inertial>
 	</link>
+	<!-- IMU reference
+	<link name="camera_gyro_frame"/> -->
 </robot>

File: catkin_ws/src/prototipo1/urdf/joints.xacro (robot description, xacro)
@@ -64,6 +64,6 @@
 	<joint name="imu_joint" type="fixed">
 		<parent link="camera_link" />
-		<child link="camera_imu_optical_frame" />
-		<origin xyz="0 0 0" rpy="0 0 0" />
+		<child link="camera_gyro_frame" />
+		<origin xyz="0 0 0" rpy="${PI} 0 0" />
 	</joint> -->
 </robot>
