Commit message: Fix link name in joints.xacro

File: catkin_ws/src/prototipo1/urdf/joints.xacro (robot description, xacro)
@@ -9,5 +9,5 @@
 		<joint name="base_support_joint" type="fixed">
 				<parent link="base_link"/>
-				<parent link="support"/>
+				<parent link="vertical_support_link"/>
 				<origin xyz="0.205 0 ${(1/2)*BASE_THICKNESS}" rpy="0 0 0"/>
 		</joint>

Commit message: Making modifications to config controllers

File: catkin_ws/src/prototipo1/urdf/joints.xacro (robot description, xacro)
@@ -13,5 +13,5 @@
 		<parent link="base_link" />
 		<child link="chassi_link" />
-		<origin xyz="-0.001 0 0" rpy="0 0 0" />
+		<origin xyz="0 0 0" rpy="0 0 0" />
 	</joint>
 	<joint name="base_support_joint" type="fixed">

Commit message: Updating xacro file to insert transmissions and actuators

File: catkin_ws/src/prototipo1/urdf/joints.xacro (robot description, xacro)
@@ -22,12 +22,20 @@
 	<!-- By the conventions of ROS urdf/tf, left side is positive y axis, as so, side parameter is 1 if left, -1 if right-->
 	<xacro:macro name="wheel_joint" params="position_prefix side">
-		<joint name="${position_prefix}_wheel_joint" type="continuous">
-			<parent link="base_link" />
-			<child link="${position_prefix}_wheel_link" />
-			<!-- Adjust position based on the side that's on-->
-			<origin xyz="0 ${side*BASE_WHEEL_DIST} 0" rpy="${-(1/2)*PI*side} 0 0" />
-			<!-- Positive around counterclockwise z-axis -->
-			<axis xyz="0 0 ${side}" />
-		</joint>
+		<transmission name="${position_prefix}_wheel_joint_trans">
+			<type> transmission_interface/SimpleTransmission </type>
+			<joint name="${position_prefix}_wheel_joint" type="continuous">
+				<parent link="base_link" />
+				<child link="${position_prefix}_wheel_link" />
+				<!-- Adjust position based on the side that's on-->
+				<origin xyz="0 ${side*BASE_WHEEL_DIST} 0" rpy="${-(1/2)*PI*side} 0 0" />
+				<!-- Positive around counterclockwise z-axis -->
+				<axis xyz="0 0 ${side}" />
+				<hardwareInterface> hardware_interface/VelocityJointInterface </hardwareInterface>
+			</joint>
+			<actuator name="${position_prefix}_wheel_joint_motor">
+				<hardwareInterface> hardware_interface/VelocityJointInterface </hardwareInterface>
+				<mechanicalReduction>50</mechanicalReduction>
+			</actuator>
+		</transmission>
 	</xacro:macro>
 	<!-- Define actual joints-->

Commit message: Updating xacro file to insert transmissions and actuators

File: catkin_ws/src/prototipo1/urdf/joints.xacro (robot description, xacro)
@@ -22,7 +22,5 @@
 	<!-- By the conventions of ROS urdf/tf, left side is positive y axis, as so, side parameter is 1 if left, -1 if right-->
 	<xacro:macro name="wheel_joint" params="position_prefix side">
-		<transmission name="${position_prefix}_wheel_joint_trans">
-			<type> transmission_interface/SimpleTransmission </type>
-			<joint name="${position_prefix}_wheel_joint" type="continuous">
+		<joint name="${position_prefix}_wheel_joint" type="continuous">
 				<parent link="base_link" />
 				<child link="${position_prefix}_wheel_link" />
@@ -31,4 +29,11 @@
 				<!-- Positive around counterclockwise z-axis -->
 				<axis xyz="0 0 ${side}" />
+				<hardwareInterface> hardware_interface/VelocityJointInterface </hardwareInterface>
+			</joint>
+	</xacro:macro>
+	<xacro:macro name="transmission_wheel" params="position_prefix">
+		<transmission name="${position_prefix}_wheel_joint_trans">
+			<type> transmission_interface/SimpleTransmission </type>
+			<joint name="${position_prefix}_wheel_joint" type="continuous">
 				<hardwareInterface> hardware_interface/VelocityJointInterface </hardwareInterface>
 			</joint>
@@ -42,4 +47,6 @@
 	<xacro:wheel_joint position_prefix="left" side="1" />
 	<xacro:wheel_joint position_prefix="right" side="-1" />
+	<xacro:transmission_wheel position_prefix="left" />
+	<xacro:transmission_wheel position_prefix="right" />
 	<!-- Joint to connect lidar to base -->
 	<joint name="base_lidar_joint" type="fixed">

Commit message: Fixing laser orientation in reference to robot model

File: catkin_ws/src/prototipo1/urdf/joints.xacro (robot description, xacro)
@@ -5,5 +5,5 @@
 	<!-- Joint distance parameters -->
 	<xacro:property name="CAMERA_HEIGHT" value="${(4/5)*SUPPORT_THICKNESS}" />
-	<xacro:property name="BASE_LIDAR_DIST" value="0.2" />
+	<xacro:property name="BASE_LIDAR_DIST" value="0.247" />
 	<xacro:property name="BASE_WHEEL_DIST" value="0.28" />
 	<xacro:property name="BASE_SUPPORT_DIST" value="0.205" />
@@ -53,5 +53,5 @@
 		<parent link="base_link" />
 		<child link="lidar_link" />
-		<origin xyz="${BASE_LIDAR_DIST} 0 ${(1/2)*CHASSI_THICKNESS}" rpy="0 0 0" />
+		<origin xyz="${BASE_LIDAR_DIST} 0 ${(1/2)*CHASSI_THICKNESS}" rpy="0 0 ${PI}" />
 	</joint>
 	<!-- Joint to connect camera to support -->

Commit message: Trying to fix IMU position

File: catkin_ws/src/prototipo1/urdf/joints.xacro (robot description, xacro)
@@ -4,5 +4,5 @@
 	<xacro:property name="PI" value="3.14159" />
 	<!-- Joint distance parameters -->
-	<xacro:property name="CAMERA_HEIGHT" value="${(4/5)*SUPPORT_THICKNESS}" />
+	<xacro:property name="CAMERA_HEIGHT" value="0.185" />
 	<xacro:property name="BASE_LIDAR_DIST" value="0.247" />
 	<xacro:property name="BASE_WHEEL_DIST" value="0.28" />
@@ -55,15 +55,9 @@
 		<origin xyz="${BASE_LIDAR_DIST} 0 ${(1/2)*CHASSI_THICKNESS}" rpy="0 0 ${PI}" />
 	</joint>
-	<!-- Joint to connect camera to support -->
-	<joint name="vertical_support_camera_joint" type="fixed">
-		<parent link="vertical_support_link" />
+	<!-- Joint to connect camera to base-->
+	<joint name="camera_joint" type="fixed">
+		<parent link="chassi_link" />
 		<child link="camera_link" />
-		<origin xyz="${SUPPORT_RADIUS} 0 ${CAMERA_HEIGHT}" rpy="${PI/2} 0 0" />
+		<origin xyz="${BASE_LIDAR_DIST} 0 ${CAMERA_HEIGHT}" rpy="0 0 0" />
 	</joint>
-	<!-- Connect unified IMU link to camera_link
-	<joint name="imu_joint" type="fixed">
-		<parent link="camera_link" />
-		<child link="camera_gyro_frame" />
-		<origin xyz="0 0 0" rpy="${PI} 0 0" />
-	</joint> -->
 </robot>
